File: VoidSwitch/VoidSwitch.kicad_pcb (KiCad board)
At the start: 2 copper layers, 22.4 x 22.3 mm, 7 parts, among them J1 IPS-4102T-01Y900, J2 IPS-4102T-01Y900, J3 IPS-4102T-01Y900, J4 IPS-4102T-01Y900, U1 DRV5032FBDBZR

Commit message: syncing
Parts:
- added ?: , , F.Cu at (144.9, 92.2)
- added GND: TestPoint, TestPoint:TestPoint_Loop_D3.80mm_Drill2.0mm, B.Cu at (145.1, 99.9)
- D1: footprint LED_SMD:LED_WS2812B_PLCC4_5.0x5.0mm_P3.2mm -> LED_SMD:LED_SK6812_EC15_1.5x1.5mm
- moved D1 2.77 mm to (148.4, 96.0), turned to 90 degrees
- moved DIN 1.45 mm to (140.4, 96.3), turned to -90 degrees
- moved DOUT 1.36 mm to (156.4, 97.1), turned to 90 degrees
- moved +5V 1.35 mm to (148.0, 104.7), turned to 0 degrees
- moved GPIO 1.31 mm to (148.9, 88.6), turned to 180 degrees
- moved HE 0.54 mm to (151.6, 99.8), turned to 180 degrees
- renumbered J3 to +5V, J1 to DIN, J2 to DOUT, J4 to GPIO, U1 to HE
Routing:
- net +5V: track 28.4 -> 15.0 mm
- net /GPIO: track 23.5 -> 12.9 mm
- net /DOUT: track 14.5 -> 11.0 mm
- net /DIN: track 11.5 -> 9.54 mm
Other:
- board size 22.4 x 22.3 mm -> 18 x 18.1 mm
