File: VoidSwitch/VoidSwitch.kicad_sch (KiCad schematic)
At the start: 7 parts, among them J1 IPS-4102T-01Y900, J2 IPS-4102T-01Y900, J3 IPS-4102T-01Y900, J4 IPS-4102T-01Y900, U1 DRV5032FBDBZR

Commit message: syncing
Parts:
- added TP1: TestPoint, TestPoint:TestPoint_Loop_D3.80mm_Drill2.0mm, symbol Connector:TestPoint
- D1: footprint LED_SMD:LED_WS2812B_PLCC4_5.0x5.0mm_P3.2mm -> LED_SMD:LED_SK6812_EC15_1.5x1.5mm
- J1, J2, J3, J4: footprint CONN2_IPS-4102T_IRE -> PressureConnectors:CONN2_IPS-4102T_IRE
Connections:
- net GND: now also TP1.1
Changed lines of the file:
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@@
       (effects (font (size 1.524 1.524)) (justify left))
     )
-    (property "Footprint" "CONN2_IPS-4102T_IRE" (at 205.74 100.33 0)
+    (property "Footprint" "PressureConnectors:CONN2_IPS-4102T_IRE" (at 205.74 100.33 0)
       (effects (font (size 1.27 1.27) italic) hide)
     )
@@
     )
   )
+  (symbol (lib_id "power:GND") (at 120.65 69.85 0) (unit 1)
+    (in_bom yes) (on_board yes) (dnp no) (fields_autoplaced)
+    (property "Reference" "#PWR08" (at 120.65 76.2 0)
+      (effects (font (size 1.27 1.27)) hide)
+    )
+    (property "Value" "GND" (at 120.65 74.93 0)
+      (effects (font (size 1.27 1.27)))
+    )
+    (property "Footprint" "" (at 120.65 69.85 0)
+      (effects (font (size 1.27 1.27)) hide)
+    )
+    (property "Datasheet" "" (at 120.65 69.85 0)
+      (effects (font (size 1.27 1.27)) hide)
+    )
+    (pin "1")
+    (instances
+      (project "VoidSwitch"
+        (path "/3da64edd-4e61-4fd4-8a88-700b3c55c60c"
+          (reference "#PWR08") (unit 1)
+        )
+      )
+    )
+  )
   (symbol (lib_id "power:+5V") (at 102.87 71.12 0) (unit 1)
     (in_bom yes) (on_board yes) (dnp no) (fields_autoplaced)
@@
       (effects (font (size 1.524 1.524)) (justify left))
     )
-    (property "Footprint" "CONN2_IPS-4102T_IRE" (at 205.74 80.01 0)
+    (property "Footprint" "PressureConnectors:CONN2_IPS-4102T_IRE" (at 205.74 80.01 0)
       (effects (font (size 1.27 1.27) italic) hide)
     )
@@
       (effects (font (size 1.27 1.27)))
     )
-    (property "Footprint" "LED_SMD:LED_WS2812B_PLCC4_5.0x5.0mm_P3.2mm" (at 161.29 74.93 0)
+    (property "Footprint" "LED_SMD:LED_SK6812_EC15_1.5x1.5mm" (at 161.29 74.93 0)
       (effects (font (size 1.27 1.27)) (justify left top) hide)
     )
@@
       (effects (font (size 1.524 1.524)) (justify left))
     )
-    (property "Footprint" "CONN2_IPS-4102T_IRE" (at 205.74 90.17 0)
+    (property "Footprint" "PressureConnectors:CONN2_IPS-4102T_IRE" (at 205.74 90.17 0)
       (effects (font (size 1.27 1.27) italic) hide)
     )
@@
       (effects (font (size 1.524 1.524)) (justify left))
     )
-    (property "Footprint" "CONN2_IPS-4102T_IRE" (at 205.74 69.85 0)
+    (property "Footprint" "PressureConnectors:CONN2_IPS-4102T_IRE" (at 205.74 69.85 0)
       (effects (font (size 1.27 1.27) italic) hide)
     )
@@
         )
       )
+    )
+  )
+  (symbol (lib_id "Connector:TestPoint") (at 120.65 69.85 0) (unit 1)
+    (in_bom yes) (on_board yes) (dnp no) (fields_autoplaced)
+    (property "Reference" "TP1" (at 123.19 65.278 0)
+      (effects (font (size 1.27 1.27)) (justify left))
+    )
+    (property "Value" "TestPoint" (at 123.19 67.818 0)
+      (effects (font (size 1.27 1.27)) (justify left))
+    )
+    (property "Footprint" "TestPoint:TestPoint_Loop_D3.80mm_Drill2.0mm" (at 125.73 69.85 0)
+      (effects (font (size 1.27 1.27)) hide)
+    )
+    (property "Datasheet" "~" (at 125.73 69.85 0)
+      (effects (font (size 1.27 1.27)) hide)
+    )
+    (pin "1")
+    (instances
+      (project "VoidSwitch"
+        (path "/3da64edd-4e61-4fd4-8a88-700b3c55c60c"
+          (reference "TP1") (unit 1)
+        )
+      )
